File: kicad/la4440.kicad_pcb (KiCad board)
At the start: 2 copper layers, 90 x 70 mm, 45 parts, among them J1 LINE IN L/GND/R, J2 VOLUME / CONTROL, J3 MUTE SWITCH, J4 DC IN +/-, J5 SPEAKER L, J6 SPEAKER R, J7 HEATSINK GND (M3 lug), Q1 2N3904, Q2 2N5401, U1 LA4440

Commit message: Label every jack and terminal pin on the silkscreen; drop the README 'not verified' section
J1 L/G/R, J2 Li/Lw/Ri/Rw/G/MC, J3 SW, J4 and speaker +/-. Q2 emitter link
is now a locked pre-routed stub (gen_pcb.py) instead of a post-route patch,
so a rebuild no longer depends on where freerouting lands. DRC 0 with parity.
Parts:
- moved C1 2.50 mm to (75.0, 76.0)
- moved C13 2.50 mm to (60.5, 70.0)
- moved C14 2.50 mm to (60.5, 87.0)
- moved R3 2.50 mm to (59.7, 64.0)
- moved R4 2.50 mm to (59.7, 80.5)
- moved R5 2.50 mm to (59.7, 60.5)
- moved R6 2.50 mm to (59.7, 77.0)
Routing:
- net /GND: track 330.5 -> 365.1 mm
- net /VCC: track 150.8 -> 164.7 mm, vias 0 -> 1
- net /ZB1: track 16.9 -> 28.9 mm
- net /ZB2: track 16.5 -> 27.2 mm
- net /WL: track 19.2 -> 24.4 mm
- net /IN2: track 34.6 -> 39.1 mm
- net /PB: track 33.6 -> 37.9 mm
- net /OUT1: track 41.3 -> 44.3 mm
- net /MUTE: track 76.2 -> 73.6 mm
- net /WR: track 17.5 -> 20.0 mm
- net /IN1: track 17.0 -> 14.5 mm
- net /Q1B: track 41.3 -> 43.3 mm
- net /W1: track 14.9 -> 15.6 mm
- net /MV: track 48.4 -> 49.0 mm
Other:
- board text added: "+"
- board text added: "-"
- board text added: "G"
- board text added: "Li"
- board text added: "Lw"
- board text added: "MC"
- board text added: "R"
- board text added: "Ri"
- board text added: "Rw"
- board text added: "SW"
