File: kicad/panel/la4440-panel-2up.kicad_pcb (KiCad board)
At the start: 2 copper layers, 90 x 142.1 mm, 118 parts, among them J1 LINE IN L/GND/R, J2 VOLUME / CONTROL, J3 MUTE SWITCH, J4 DC IN +/-, J5 SPEAKER L, J6 SPEAKER R, J7 HEATSINK GND (M3 lug), Q1 2N3904, Q2 2N5401, U1 LA4440

Commit message: Label every jack and terminal pin on the silkscreen; drop the README 'not verified' section
J1 L/G/R, J2 Li/Lw/Ri/Rw/G/MC, J3 SW, J4 and speaker +/-. Q2 emitter link
is now a locked pre-routed stub (gen_pcb.py) instead of a post-route patch,
so a rebuild no longer depends on where freerouting lands. DRC 0 with parity.
Parts:
- removed the C1 at (22.5, 98.1)
- removed the C1 at (22.5, 26.0)
- removed the C13 at (8.00, 92.1)
- removed the C13 at (8.00, 20.0)
- removed the C14 at (8.00, 37.0)
- removed the C14 at (8.00, 109.1)
- removed the R3 at (7.20, 14.0)
- removed the R3 at (7.20, 86.1)
- removed the R4 at (7.20, 102.6)
- removed the R4 at (7.20, 30.5)
- removed the R5 at (7.20, 82.6)
- removed the R5 at (7.20, 10.5)
- removed the R6 at (7.20, 99.1)
- removed the R6 at (7.20, 27.0)
- added C1: 47u 50V, Capacitor_THT:CP_Radial_D8.0mm_P3.50mm, F.Cu at (25.0, 98.1)
- added C1: 47u 50V, Capacitor_THT:CP_Radial_D8.0mm_P3.50mm, F.Cu at (25.0, 26.0)
- added C13: 47u 50V, Capacitor_THT:CP_Radial_D8.0mm_P3.50mm, F.Cu at (10.5, 20.0)
- added C13: 47u 50V, Capacitor_THT:CP_Radial_D8.0mm_P3.50mm, F.Cu at (10.5, 92.1)
- added C14: 47u 50V, Capacitor_THT:CP_Radial_D8.0mm_P3.50mm, F.Cu at (10.5, 109.1)
- added C14: 47u 50V, Capacitor_THT:CP_Radial_D8.0mm_P3.50mm, F.Cu at (10.5, 37.0)
- added R3: 10k, Custom:R_Axial_1206, F.Cu at (9.70, 14.0)
- added R3: 10k, Custom:R_Axial_1206, F.Cu at (9.70, 86.1)
- added R4: 10k, Custom:R_Axial_1206, F.Cu at (9.70, 102.6)
- added R4: 10k, Custom:R_Axial_1206, F.Cu at (9.70, 30.5)
- added R5: 5.6k, Custom:R_Axial_1206, F.Cu at (9.70, 10.5)
- added R5: 5.6k, Custom:R_Axial_1206, F.Cu at (9.70, 82.6)
- added R6: 5.6k, Custom:R_Axial_1206, F.Cu at (9.70, 99.1)
- added R6: 5.6k, Custom:R_Axial_1206, F.Cu at (9.70, 27.0)
Routing:
- net Board_0-/GND: track 330.5 -> 365.1 mm
- net Board_1-/GND: track 330.5 -> 365.1 mm
- net Board_0-/VCC: track 150.8 -> 164.7 mm, vias 0 -> 1
- net Board_1-/VCC: track 150.8 -> 164.7 mm, vias 0 -> 1
- net Board_1-/ZB1: track 16.9 -> 28.9 mm
- net Board_0-/ZB1: track 16.9 -> 28.9 mm
- net Board_1-/ZB2: track 16.5 -> 27.2 mm
- net Board_0-/ZB2: track 16.5 -> 27.2 mm
- net Board_1-/WL: track 19.2 -> 24.4 mm
- net Board_0-/WL: track 19.2 -> 24.4 mm
- net Board_0-/IN2: track 34.6 -> 39.1 mm
- net Board_1-/IN2: track 34.6 -> 39.1 mm
- net Board_0-/PB: track 33.6 -> 37.9 mm
- net Board_1-/PB: track 33.6 -> 37.9 mm
- net Board_1-/OUT1: track 41.3 -> 44.3 mm
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Other:
- board text added: "+"
- board text added: "-"
- board text added: "G"
- board text added: "Li"
- board text added: "Lw"
- board text added: "MC"
- board text added: "R"
- board text added: "Ri"
- board text added: "Rw"
- board text added: "SW"
